Commit message: New urdf

File: Matlab/urdf/robot.urdf (robot description, URDF)
Before this commit: robot Eden, 6 links, 5 joints
Links:
- removed link world
- added link camera, mass 0.000135; collision mesh filename=package://meshes/camera.stl; visual mesh filename=package://meshes/camera.stl
- added link origin
- added link target, mass 3.375e-05; collision mesh filename=package://meshes/target.stl; visual mesh filename=package://meshes/target.stl
- link hand: mass 0.301016 -> 0.300847; geometry collision mesh filename=package://meshes/ax_12w.stl; collision mesh filename=package://meshes/big_gear_wrist.stl
Joints:
- added joint camera: type fixed, parent hand, child camera, origin xyz=0.0560004 0.08 -0.0105 rpy=1.5708 3.04281e-32 8.99294e-30, axis 0 0 1, limit effort=1 velocity=20
- added joint target: type fixed, parent hand, child target, origin xyz=0.000500416 0.23624 -0.0105 rpy=1.5708 1.5708 0, axis 0 0 1, limit effort=1 velocity=20
- joint fixed: parent world -> origin

File: Python/urdf/robot.urdf (robot description, URDF)
Before this commit: robot Eden, 6 links, 5 joints
Links:
- removed link reference
- added link camera, mass 0.000135; collision mesh filename=package:///camera.stl; visual mesh filename=package:///camera.stl
- added link origin
- added link target, mass 3.375e-05; collision mesh filename=package:///target.stl; visual mesh filename=package:///target.stl
- link hand: mass 0.301016 -> 0.300847; geometry collision mesh filename=package:///ax_12w.stl; collision mesh filename=package:///big_gear_wrist.stl
Joints:
- added joint camera: type fixed, parent hand, child camera, origin xyz=0.0560004 0.08 -0.0105 rpy=1.5708 3.04281e-32 8.99294e-30, axis 0 0 1, limit effort=1 velocity=20
- added joint target: type fixed, parent hand, child target, origin xyz=0.000500416 0.23624 -0.0105 rpy=1.5708 1.5708 0, axis 0 0 1, limit effort=1 velocity=20
- joint fixed: parent reference -> origin

Commit message: inverse kinematics correction

File: Matlab/urdf/robot.urdf (robot description, URDF)
Before this commit: robot onshape, 8 links, 7 joints
Links:
- link base: geometry collision mesh filename=package://meshes/adapteur.stl; collision mesh filename=package://meshes/cover.stl
- link hip: geometry collision mesh filename=package://meshes/big_gear_pelvis.stl; collision mesh filename=package://meshes/fixing_base_tree.stl

File: Python/urdf/robot.urdf (robot description, URDF)
Before this commit: robot onshape, 8 links, 7 joints
Links:
- link base: geometry collision mesh filename=package:///adapteur.stl; collision mesh filename=package:///cover.stl
- link hip: geometry collision mesh filename=package:///big_gear_pelvis.stl; collision mesh filename=package:///fixing_base_tree.stl

Commit message: Report management

File: Matlab/urdf/robot.urdf (robot description, URDF)
Before this commit: robot onshape, 8 links, 7 joints
Links:
- link base: mass 1.76245 -> 1.26177; geometry collision mesh filename=package:///adapteur.stl; collision mesh filename=package:///cover.stl
- link camera: geometry collision mesh filename=package:///camera.stl; visual mesh filename=package:///camera.stl
- link hand: mass 0.300847 -> 0.16977; geometry collision mesh filename=package:///ax_12w.stl; collision mesh filename=package:///big_gear_wrist.stl
- link hip: mass 0.680307 -> 0.468773; geometry collision mesh filename=package:///big_gear_pelvis.stl; collision mesh filename=package:///fixing_base_tree.stl
- link humerus: mass 0.410438 -> 0.390303; geometry collision mesh filename=package:///arm_elbow.stl; collision mesh filename=package:///arm_elbow.stl
- link radius: mass 0.416076 -> 0.380955; geometry collision mesh filename=package:///arm_elbow.stl; collision mesh filename=package:///arm_elbow.stl
- link target: geometry collision mesh filename=package:///target.stl; visual mesh filename=package:///target.stl

File: Python/urdf/robot.urdf (robot description, URDF)
Before this commit: robot onshape, 8 links, 7 joints
Links:
- link base: mass 1.76245 -> 1.26177
- link hand: mass 0.300847 -> 0.16977
- link hip: mass 0.680307 -> 0.468773
- link humerus: mass 0.410438 -> 0.390303
- link radius: mass 0.416076 -> 0.380955

Commit message: urdf correction

File: Matlab/urdf/robot.urdf (robot description, URDF)
Before this commit: robot onshape, 8 links, 7 joints
Links:
- link base: geometry collision mesh filename=package://meshes/adapteur.stl; collision mesh filename=package://meshes/bottom.stl
- link camera: geometry collision mesh filename=package://meshes/camera.stl; visual mesh filename=package://meshes/camera.stl
- link hand: mass 0.16977 -> 0.191614; geometry collision mesh filename=package://meshes/ax_12w.stl; collision mesh filename=package://meshes/big_gear_wrist.stl
- link hip: geometry collision mesh filename=package://meshes/big_gear_pelvis.stl; collision mesh filename=package://meshes/fixing_base_tree.stl
- link humerus: geometry collision mesh filename=package://meshes/big_gear_shoulder.stl; collision mesh filename=package://meshes/fixing_shoulder_tree.stl
- link radius: geometry collision mesh filename=package://meshes/big_gear_elbow.stl; collision mesh filename=package://meshes/motor_link_xl.stl
- link target: geometry collision mesh filename=package://meshes/target.stl; visual mesh filename=package://meshes/target.stl
Joints:
- joint camera: origin xyz=0.0560004 0.08 -0.0105 rpy=1.5708 3.04281e-32 8.99294e-30 -> xyz=0.0560004 0.08 -0.0105 rpy=1.5708 -1.70787e-28 1.9082e-16
- joint elbow: origin xyz=1.44329e-14 0.16 -0.042 rpy=-3.14159 1.78606e-16 1.5708 -> xyz=1.38778e-17 0.16 -0.042 rpy=3.14159 1.78606e-16 1.5708
- joint pelvis: origin xyz=-0.06 4.33681e-18 0.069 rpy=-3.14159 5.66994e-31 -1.5708 -> xyz=-0.06 6.93889e-18 0.069 rpy=3.14159 -1.19271e-28 -1.5708
- joint shoulder: origin xyz=-0.018 -1.04361e-14 -0.116 rpy=-1.5708 -2.22045e-16 1.5708 -> xyz=-0.018 2.08167e-17 -0.116 rpy=-1.5708 7.82376e-14 1.5708
- joint wrist: origin xyz=4.44089e-15 0.155 -0.014125 rpy=3.18115e-24 -3.87963e-29 -7.26676e-14 -> xyz=-4.77396e-15 0.155 -0.014125 rpy=2.22045e-16 -2.15076e-25 -4.74015e-14

File: Python/urdf/robot.urdf (robot description, URDF)
Before this commit: robot onshape, 8 links, 7 joints
Links:
- link base: geometry collision mesh filename=package:///adapteur.stl; collision mesh filename=package:///bottom.stl
- link hand: mass 0.16977 -> 0.191614; geometry collision mesh filename=package:///ax_12w.stl; collision mesh filename=package:///big_gear_wrist.stl
- link humerus: geometry collision mesh filename=package:///big_gear_shoulder.stl; collision mesh filename=package:///fixing_shoulder_tree.stl
- link radius: geometry collision mesh filename=package:///big_gear_elbow.stl; collision mesh filename=package:///motor_link_xl.stl
Joints:
- joint camera: origin xyz=0.0560004 0.08 -0.0105 rpy=1.5708 3.04281e-32 8.99294e-30 -> xyz=0.0560004 0.08 -0.0105 rpy=1.5708 -1.70787e-28 1.9082e-16
- joint elbow: origin xyz=1.44329e-14 0.16 -0.042 rpy=-3.14159 1.78606e-16 1.5708 -> xyz=1.38778e-17 0.16 -0.042 rpy=3.14159 1.78606e-16 1.5708
- joint pelvis: origin xyz=-0.06 4.33681e-18 0.069 rpy=-3.14159 5.66994e-31 -1.5708 -> xyz=-0.06 6.93889e-18 0.069 rpy=3.14159 -1.19271e-28 -1.5708
- joint shoulder: origin xyz=-0.018 -1.04361e-14 -0.116 rpy=-1.5708 -2.22045e-16 1.5708 -> xyz=-0.018 2.08167e-17 -0.116 rpy=-1.5708 7.82376e-14 1.5708
- joint wrist: origin xyz=4.44089e-15 0.155 -0.014125 rpy=3.18115e-24 -3.87963e-29 -7.26676e-14 -> xyz=-4.77396e-15 0.155 -0.014125 rpy=2.22045e-16 -2.15076e-25 -4.74015e-14

Commit message: rename stl

File: Matlab/urdf/robot.urdf (robot description, URDF)
Before this commit: robot onshape, 8 links, 7 joints
Links:
- link hip: geometry collision mesh filename=package://meshes/big_gear_pelvis.stl; collision mesh filename=package://meshes/fixing_base_tree.stl

File: Python/urdf/robot.urdf (robot description, URDF)
Before this commit: robot onshape, 8 links, 7 joints
Links:
- link hip: geometry collision mesh filename=package:///big_gear_pelvis.stl; collision mesh filename=package:///fixing_base_tree.stl
